File: RPI-RP2040-MINIMAL_R3-S1.kicad_pcb (KiCad board)
At the start: 2 copper layers, 65 x 46.7 mm, 34 parts, among them J1 Conn_01x03_Socket, J3 Conn_01x04_Pin, J4 Conn_01x04_Socket, P1 USB_C_Plug_USB2.0, U1 NCP1117ST33T3G, U2 W25Q128JVSIQ, U3 RP2040, X1 12MHz

Commit message: Rounding
Routing:
- net /BRIDGE_USBD-: track 15.9 -> 17.9 mm
- net +1V1: track 18.1 -> 17.5 mm
Other:
- board text added: "C G D"
- board text removed: "CLK GND SWD"
Changed lines of the file:
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@@
 				(font
 					(size 1.27 1.27)
+					(thickness 0.15)
 				)
 			)
@@
 				(font
 					(size 1.27 1.27)
+					(thickness 0.15)
 				)
 			)
@@
 		)
 	)
+	(gr_rect
+		(start 65 95.25)
+		(end 75 105.25)
+		(stroke
+			(width 0.12)
+			(type default)
+		)
+		(fill no)
+		(layer "F.SilkS")
+	)
 	(gr_line
 		(start 50.5 61.7517)
@@
 		(layer "Edge.Cuts")
 	)
-	(gr_text "CLK GND SWD"
-		(at 106 103.5 0)
+	(gr_text "C G D"
+		(at 105.5 106.25 0)
 		(layer "F.SilkS")
 		(effects
 			(font
-				(size 0.3 0.3)
+				(size 0.8 0.8)
 			)
 			(justify left bottom)
@@
 	)
 	(gr_text "DEBUG"
-		(at 106 103 0)
+		(at 105.75 103.25 0)
 		(layer "F.SilkS")
 		(effects
 			(font
-				(size 0.75 0.75)
+				(size 0.8 0.8)
 			)
 			(justify left bottom)
@@
 	)
 	(segment
-		(start 100.265 104.424274)
-		(end 100.265 103.745)
-		(width 0.2)
-		(layer "F.Cu")
-		(net "+1V1")
-	)
-	(segment
 		(start 100.755 98.245)
 		(end 100.365 98.245)
@@
 	)
 	(segment
+		(start 100.39 105.103495)
+		(end 100.265 104.978495)
+		(width 0.15)
+		(layer "F.Cu")
+		(net "+1V1")
+	)
+	(segment
 		(start 101.465 96.945)
 		(end 101.465 97.535)
@@
 	)
 	(segment
+		(start 100.265 104.978495)
+		(end 100.265 103.745)
+		(width 0.15)
+		(layer "F.Cu")
+		(net "+1V1")
+	)
+	(segment
 		(start 98.665 93.345)
 		(end 98.665 93.64)
@@
 	)
 	(segment
-		(start 100.265 103.745)
-		(end 100.265 105.103495)
-		(width 0.2)
-		(layer "F.Cu")
-		(net "+1V1")
-	)
-	(segment
 		(start 101.465 96.9075)
 		(end 101.465 96.145)
@@
 	)
 	(segment
+		(start 57.548963 68.800663)
+		(end 57.885 69.1367)
+		(width 0.8)
+		(layer "F.Cu")
+		(net "/BRIDGE_USBD-")
+	)
+	(segment
 		(start 56.290369 67.92302)
 		(end 55.862379 68.35101)
@@
 	)
 	(segment
+		(start 57.548963 67.2517)
+		(end 57.548963 68.800663)
+		(width 0.8)
+		(layer "F.Cu")
+		(net "/BRIDGE_USBD-")
+	)
+	(segment
 		(start 68.304491 69.1367)
 		(end 57.885 69.1367)
@@
 	)
 	(segment
+		(start 101.065 103.745)
+		(end 101.065 104.285736)
+		(width 0.15)
+		(layer "F.Cu")
+		(net "/SWD")
+	)
+	(segment
+		(start 103.28 104.22)
+		(end 103.97 104.22)
+		(width 0.15)
+		(layer "F.Cu")
+		(net "/SWD")
+	)
+	(segment
+		(start 103 104.5)
+		(end 103.28 104.22)
+		(width 0.15)
+		(layer "F.Cu")
+		(net "/SWD")
+	)
+	(segment
+		(start 101.279264 104.5)
+		(end 103 104.5)
+		(width 0.15)
+		(layer "F.Cu")
+		(net "/SWD")
+	)
+	(segment
+		(start 101.065 104.285736)
+		(end 101.279264 104.5)
+		(width 0.15)
+		(layer "F.Cu")
+		(net "/SWD")
+	)
+	(segment
+		(start 107.875 103.685)
+		(end 108.525 104.335)
+		(width 0.15)
+		(layer "F.Cu")
+		(net "Net-(J1-Pin_3)")
+	)
+	(segment
+		(start 104.99 104.22)
+		(end 105.525 103.685)
+		(width 0.15)
+		(layer "F.Cu")
+		(net "Net-(J1-Pin_3)")
+	)
+	(segment
+		(start 105.525 103.685)
+		(end 107.875 103.685)
+		(width 0.15)
+		(layer "F.Cu")
+		(net "Net-(J1-Pin_3)")
+	)
+	(segment
 		(start 96.265 98.145)
 		(end 80.245978 98.145)
@@
 	)
 	(segment
+		(start 100.665 103.745)
+		(end 100.665 104.31)
+		(width 0.15)
+		(layer "F.Cu")
+		(net "/SWCLK")
+	)
+	(segment
+		(start 101.574113 105.219113)
+		(end 103.977791 105.219113)
+		(width 0.15)
+		(layer "F.Cu")
+		(net "/SWCLK")
+	)
+	(segment
+		(start 100.665 104.31)
+		(end 101.574113 105.219113)
+		(width 0.15)
+		(layer "F.Cu")
+		(net "/SWCLK")
+	)
+	(segment
+		(start 104.997791 105.219113)
+		(end 105.640887 105.219113)
+		(width 0.15)
+		(layer "F.Cu")
+		(net "Net-(J1-Pin_1)")
+	)
+	(segment
+		(start 105.640887 105.219113)
+		(end 106.525 104.335)
+		(width 0.15)
+		(layer "F.Cu")
+		(net "Net-(J1-Pin_1)")
+	)
+	(segment
 		(start 88.665 91.045)
 		(end 87.765 90.145)
@@
 	)
 	(segment
-		(start 100.665 103.745)
-		(end 100.665 104.31)
-		(width 0.15)
-		(layer "F.Cu")
-		(net "/SWCLK")
-	)
-	(segment
-		(start 101.574113 105.219113)
-		(end 103.977791 105.219113)
-		(width 0.15)
-		(layer "F.Cu")
-		(net "/SWCLK")
-	)
-	(segment
-		(start 100.665 104.31)
-		(end 101.574113 105.219113)
-		(width 0.15)
-		(layer "F.Cu")
-		(net "/SWCLK")
-	)
-	(segment
-		(start 101.065 103.745)
-		(end 101.065 104.285736)
-		(width 0.15)
-		(layer "F.Cu")
-		(net "/SWD")
-	)
-	(segment
-		(start 103.28 104.22)
-		(end 103.97 104.22)
-		(width 0.15)
-		(layer "F.Cu")
-		(net "/SWD")
-	)
-	(segment
-		(start 103 104.5)
-		(end 103.28 104.22)
-		(width 0.15)
-		(layer "F.Cu")
-		(net "/SWD")
-	)
-	(segment
-		(start 101.279264 104.5)
-		(end 103 104.5)
-		(width 0.15)
-		(layer "F.Cu")
-		(net "/SWD")
-	)
-	(segment
-		(start 101.065 104.285736)
-		(end 101.279264 104.5)
-		(width 0.15)
-		(layer "F.Cu")
-		(net "/SWD")
-	)
-	(segment
 		(start 101.065 95.645)
 		(end 101.665 95.045)
@@
 		(net "/USB_D-")
 	)
-	(segment
-		(start 107.875 103.685)
-		(end 108.525 104.335)
-		(width 0.15)
-		(layer "F.Cu")
-		(net "Net-(J1-Pin_3)")
-	)
-	(segment
-		(start 104.99 104.22)
-		(end 105.525 103.685)
-		(width 0.15)
-		(layer "F.Cu")
-		(net "Net-(J1-Pin_3)")
-	)
-	(segment
-		(start 105.525 103.685)
-		(end 107.875 103.685)
-		(width 0.15)
-		(layer "F.Cu")
-		(net "Net-(J1-Pin_3)")
-	)
-	(segment
-		(start 104.997791 105.219113)
-		(end 105.640887 105.219113)
-		(width 0.15)
-		(layer "F.Cu")
-		(net "Net-(J1-Pin_1)")
-	)
-	(segment
-		(start 105.640887 105.219113)
-		(end 106.525 104.335)
-		(width 0.15)
-		(layer "F.Cu")
-		(net "Net-(J1-Pin_1)")
-	)
 	(zone
 		(net "/BRIDGE_VBUS")
@@
 			"1188787d-9b55-4bfb-b533-4372e5e796f7" "16541364-1a27-4dd7-b501-a1626643ce21"
 			"1a7b04c7-4b20-4338-920c-d0ed9b441c8f" "257138e0-8c02-4750-9f29-338e21e70f00"
-			"288ee3e2-d988-40b0-bd9d-ea7de64a6508" "34987f01-9a02-49e2-ae9c-1c0d6e4b879a"
-			"391d9f5c-957c-4d8b-9aeb-af80f551a1b5" "3997b664-7fbc-467e-9989-582e64dc57c5"
-			"3aa0997d-4e33-4535-ab10-8e3ba68186ec" "3d982280-7e01-40f2-92f3-356c6e73459e"
-			"61bf2c16-d640-4481-8421-19e295e17405" "6404b271-0a23-4daa-9669-2c53fca30ff3"
+			"34987f01-9a02-49e2-ae9c-1c0d6e4b879a" "391d9f5c-957c-4d8b-9aeb-af80f551a1b5"
+			"3997b664-7fbc-467e-9989-582e64dc57c5" "3aa0997d-4e33-4535-ab10-8e3ba68186ec"
+			"3d982280-7e01-40f2-92f3-356c6e73459e" "6404b271-0a23-4daa-9669-2c53fca30ff3"
 			"664a0fce-0ed9-4c2e-9395-93db82470be6" "6e100cc0-e9b3-4eb8-82b0-da4d9fa4cd20"
-			"7030e1ae-2083-4e0c-b310-6d0bb6cff4db" "71e8feaa-ad86-4fff-ad70-0ec18ffcd9e4"
-			"7dfde1cc-9cec-43cb-95df-4320f114c371" "838c6daf-b5d4-4028-91aa-34eeade1a8f6"
-			"851576c5-6fba-42c2-b7e2-4225be9d97cc" "86904204-f297-4165-9239-305653056d9d"
-			"8a055d9b-cff1-4a25-8f95-e32bc02e42eb" "8ab97694-2f58-485c-b18e-a6ffee00ea84"
-			"8d160bb8-d3f8-4df9-8f31-aee5e533a074" "8fe77c87-7bff-4a4e-b616-8c416ee26bfb"
-			"96195365-365b-4246-ad06-d37062c93fe3" "96b7201e-1eaf-4251-9978-d0425f73d9f5"
-			"9711f30b-6031-4524-9bf1-3bb795aa0915" "a3948fb9-4e5c-46f9-8916-b7fb0eadc9ee"
-			"a43971be-2932-40ed-909f-1ccc4ce9f7d0" "a83b520f-0de3-44e5-8523-669a51519cc3"
-			"a99811d5-4d79-4925-9e62-cd4e3308589b" "b8909dc5-20b3-4719-859a-3f4d6f3ab9da"
-			"c221c861-d785-4c85-b519-3ef2c23fa54d" "c66262e8-02d8-4396-8c55-98316d7eaee4"
-			"c9b54a73-55b4-4a13-b75f-a99519f7eb76" "cb457be9-a617-45d4-b949-c92afbf6ee8b"
-			"d5cff7bb-9d67-4bc1-a76e-e58f62ce7cbf" "d8e99e28-de6b-4418-94fc-b0d08fbf36d4"
-			"ec729c32-55b1-4b8e-a035-bd5ab4f56213" "f3b2230d-5e23-4f5b-a36c-16f4308f3633"
-			"f4ae312d-250b-4c3b-8e96-93bde8e4b53c"
+			"71e8feaa-ad86-4fff-ad70-0ec18ffcd9e4" "7dfde1cc-9cec-43cb-95df-4320f114c371"
+			"838c6daf-b5d4-4028-91aa-34eeade1a8f6" "851576c5-6fba-42c2-b7e2-4225be9d97cc"
+			"86904204-f297-4165-9239-305653056d9d" "8a055d9b-cff1-4a25-8f95-e32bc02e42eb"
+			"8ab97694-2f58-485c-b18e-a6ffee00ea84" "8d160bb8-d3f8-4df9-8f31-aee5e533a074"
+			"8fe77c87-7bff-4a4e-b616-8c416ee26bfb" "96195365-365b-4246-ad06-d37062c93fe3"
+			"96b7201e-1eaf-4251-9978-d0425f73d9f5" "9711f30b-6031-4524-9bf1-3bb795aa0915"
+			"a3948fb9-4e5c-46f9-8916-b7fb0eadc9ee" "a43971be-2932-40ed-909f-1ccc4ce9f7d0"
+			"a83b520f-0de3-44e5-8523-669a51519cc3" "a99811d5-4d79-4925-9e62-cd4e3308589b"
+			"b8909dc5-20b3-4719-859a-3f4d6f3ab9da" "c221c861-d785-4c85-b519-3ef2c23fa54d"
+			"c66262e8-02d8-4396-8c55-98316d7eaee4" "c9b54a73-55b4-4a13-b75f-a99519f7eb76"
+			"cb457be9-a617-45d4-b949-c92afbf6ee8b" "d5cff7bb-9d67-4bc1-a76e-e58f62ce7cbf"
+			"d8e99e28-de6b-4418-94fc-b0d08fbf36d4" "ec729c32-55b1-4b8e-a035-bd5ab4f56213"
+			"f3b2230d-5e23-4f5b-a36c-16f4308f3633" "f4ae312d-250b-4c3b-8e96-93bde8e4b53c"
 		)
 	)

Commit message: attach both sides of port
Connections:
- P1 pad B6: (no net) -> /BRIDGE_USBD+
- P1 pad B7: (no net) -> /BRIDGE_USBD-
Routing:
- net /BRIDGE_USBD+: track 14.6 -> 22.0 mm, vias 2 -> 3
- net /BRIDGE_USBD-: track 17.9 -> 23.4 mm
